File: wm61_mic_preamp/wm61_mic_preamp.sch (KiCad schematic (older format))
At the start: 18 parts, among them J1 WM60-WM61, J2 5V, J3 Out, U1 OPA2320

Commit message: changed opamp
Parts:
- U1: value OPA2320 -> MCP6L02T
Changed lines of the file:
@@
 P 6550 3350
 F 0 "U1" H 6550 3717 50  0000 C CNN
-F 1 "OPA2320" H 6550 3626 50  0000 C CNN
+F 1 "MCP6L02T" H 6550 3626 50  0000 C CNN
 F 2 "Package_SO:TSSOP-8_4.4x3mm_P0.65mm" H 6550 3350 50  0001 C CNN
 F 3 "http://www.ti.com/lit/ds/symlink/lm358.pdf" H 6550 3350 50  0001 C CNN
@@
 P 7950 3450
 F 0 "U1" H 7950 3817 50  0000 C CNN
-F 1 "OPA2320" H 7950 3726 50  0000 C CNN
+F 1 "MCP6L02T" H 7950 3726 50  0000 C CNN
 F 2 "Package_SO:TSSOP-8_4.4x3mm_P0.65mm" H 7950 3450 50  0001 C CNN
 F 3 "http://www.ti.com/lit/ds/symlink/lm358.pdf" H 7950 3450 50  0001 C CNN
